File: hardware/shrink-fit-controller/shrink-fit-controller.kicad_sch (KiCad schematic)
At the start: 0 parts

Commit message: Schematic drawn and netlist-verified; footprint adopted after de-trapping
The schematic is generated (tools/gen_sch.py), not hand-drawn, so the pinout
truth lives in one reviewed table instead of ninety mouse placements. ERC came
back 0/0, but the check that matters is the netlist-vs-expectation table: all
15 U1 nets verified on their header-position pads, and the divider and driver
chains verified by full membership, catching nothing wrong precisely because
the symbol was built from three sources first.

Two generator bugs were caught by the validation loop itself: a regex
alternation mangled the one-letter symbol names (R, C) when prefixing the
embedded library, which cascaded into all 16 ERC violations; and the netlist
parser assumed single-line format. Both fixes are in the generator. The #FLG
absence from the netlist is by design (KiCad excludes #-refs), not a failure.

The found footprint is adopted with three fixes, one of which would have been a
silent disaster: its pad "numbers" are silk NAMES, so its pad "1" is GPIO1 -
our pad 3 - and dropping it in unchanged would have landed most nets on wrong
pins with no tool complaint. Renumbered to header positions. Also 1.508/1.0
pads fail the pcbmill annulus gate at 0.164 after the 1.0->1.181 snap-up
(now 1.78/1.181 = 0.300), and one pad sat 0.04 off-grid.

Row spacing resolves to 15.24 mm; the earlier 17.78 prediction was wrong and
the footprint+photos+drawing agree three ways. Power is closed: the kit wall
wart is Class II, so the LM2596 non-isolation imports no earth bond. The only
blocker left before copper is the enclosure mounting pattern.
Parts:
- added C1: 100nF, symbol shrink-fit-controller:C
- added J1: 12V IN (kit wall wart), symbol shrink-fit-controller:CONN_02
- added J2: SSR-100DD input, symbol shrink-fit-controller:CONN_02
- added J3: Bus sense DC+/DC-, symbol shrink-fit-controller:CONN_02
- added J4: Flow switch, symbol shrink-fit-controller:CONN_02
- added J5: E-stop sense, symbol shrink-fit-controller:CONN_02
- added J6: Start button, symbol shrink-fit-controller:CONN_02
- added J7: CAN TTL (Phase 2), symbol shrink-fit-controller:CONN_04
- added J8: MAX31855 (Phase 2), symbol shrink-fit-controller:CONN_05
- added J9: INA228 I2C (Phase 2), symbol shrink-fit-controller:CONN_04
- added PS1: LM2596 module 12V->5V, symbol shrink-fit-controller:CONN_04
- added Q1: 2N3904, symbol shrink-fit-controller:Q_2N3904
- added R1: 1k, symbol shrink-fit-controller:R
- added R2: 220k, symbol shrink-fit-controller:R
- added R3: 10k, symbol shrink-fit-controller:R
- added U1: ESP32-S3 Super Mini HW-747, symbol shrink-fit-controller:ESP32-S3-SuperMini-HW747
Connections:
- new net: Q1.2 (B), R1.2
- new net +12V: J1.1, J2.1, PS1.1
- new net +3V3: J4.1, J7.1, J8.1, J9.1, U1.16 (3V3)
- new net +5V: PS1.3, U1.18 (5V)
- new net BUS_SENSE: C1.1, R2.2, R3.1, U1.3 (GPIO1)
- new net BUS_V+: J3.1, R2.1
- new net CAN_RX: J7.4, U1.7 (GPIO5)
- new net CAN_TX: J7.3, U1.6 (GPIO4)
- new net ESTOP_SENSE: J5.1, U1.9 (GPIO7)
- new net FLOW_SW: J4.2, U1.8 (GPIO6)
- new net GND: C1.2, J1.2, J3.2, J5.2, J6.2, J7.2, J8.2, J9.2, PS1.2, PS1.4, Q1.1 (E), R3.2, U1.17 (GND)
- new net SCL: J9.4, U1.11 (GPIO9)
- new net SDA: J9.3, U1.10 (GPIO8)
- new net SSR_DRV: R1.1, U1.12 (GPIO10)
- new net SSR_K: J2.2, Q1.3 (C)
- new net START_BTN: J6.1, U1.4 (GPIO2)
- new net TC_CS: J8.4, U1.13 (GPIO11)
- new net TC_MISO: J8.5, U1.15 (GPIO13)
- new net TC_SCK: J8.3, U1.14 (GPIO12)
- no-connect marks 0 -> 3
Other:
- note added: "Divider 220k/10k = 23:1 (180k not stocked). Calibrate with testrig 'cal <V>'. C1 is not optional: sensing beside a kW oscillator (R-11)."
- note added: "GND IS DC-. The controller floats with the bus (SR-11 bond withdrawn). No USB while energised; no earthed scope ground clip - differential probe only."
- note added: "GPIO3 reserved: Stage-4 encoder."
- note added: "J4 flow: switch to 3V3, firmware INPUT_PULLDOWN, active high = flow proven. J5/J6: contacts to GND, INPUT_PULLUP, active low."
- note added: "Phase 2 headers J7/J8/J9: footprints reserved, unpopulated. CAN stack (ADUM1201 + B0505S + SN65HVD230) is off-board - isolation required. INA228 shunt value is a PLACEHOLDER until VR-11 four-wire cal."
- note added: "SSR-100DD input 3-32V, fed from +12V; Q1 low-side. GPIO10 delivers the voltage STEP (CR-05) - CAN sets bus volts, never enables output."
- note added: "WIRE BY PIN NAME, NEVER BY NUMBER. U1 numbers are header positions: GPIO1 = pin 3, GPIO10 (SSR drive) = pin 12. Verify pads in the .kicad_pcb after layout."
